File: skrh-switch-breakout.kicad_pcb (KiCad board)
At the start: 2 copper layers, 0 parts

Commit message: add breakout for left side
Parts:
- added D1: 1N4148, Keebrary:Diode_D_SOD-123_Silkless_Reversible, F.Cu at (56.3, 41.5)
- added D2: 1N4148, Keebrary:Diode_D_SOD-123_Silkless_Reversible, F.Cu at (58.0, 39.9)
- added D3: 1N4148, Keebrary:Diode_D_SOD-123_Silkless_Reversible, F.Cu at (61.9, 54.7)
- added D4: 1N4148, Keebrary:Diode_D_SOD-123_Silkless_Reversible, F.Cu at (64.2, 38.9)
- added D5: 1N4148, Keebrary:Diode_D_SOD-123_Silkless_Reversible, F.Cu at (67.4, 54.7)
- added H1: Hole, Keebrary:MountingHole_2.3mm_M2_Threaded_ISO14580_Pad, F.Cu at (55.5, 53.9)
- added H2: Hole, Keebrary:MountingHole_2.3mm_M2_Threaded_ISO14580_Pad, F.Cu at (69.6, 39.7)
- added S1: SW_MultiDirectional_4DCP_SKRHACE010, Keebrary:SW_MultiDirectional_4DCP_SKRHACE010_SMD_7.5x7.5mm_Breakout, F.Cu at (62.5, 46.8)
- added kibuzzard-63DE04E8: G***, kibuzzard-63DE04E8, F.Cu at (67.1, 42.4)
Routing:
- net COMMON: track 0.00 -> 39.7 mm
- net PUSH: track 0.00 -> 20.1 mm
- net C_LEFT: track 0.00 -> 15.2 mm
- net B_RIGHT: track 0.00 -> 14.6 mm
- net D_DOWN: track 0.00 -> 12.6 mm
- net A_UP: track 0.00 -> 10.5 mm
Other:
- board outline added: 19 x 19.1 mm
- board text added: "D1"
- board text added: "D2"
- board text added: "D3"
- board text added: "D4"
- board text added: "D5"
- board text added: "SKRH Breakout (L)"
